Commit message: Seperate ft-300 coupling from sensor

File: robotiq_description/urdf/robotiq_ft_300/robotiq_ft_300_macro.xacro (robot description, xacro)
@@ -6,35 +6,5 @@
     <xacro:read_model_data
       visual_parameters_file="${visual_parameters_file}"/>
-    <!-- Link representing the FT300 mounting plate for Universal Robots -->
-    <link name="${prefix}mounting_plate">
-      <inertial>
-        <origin xyz="0.00227643166121317 -0.00163641909670073 -0.000186465195632485" rpy="0 0 0" />
-        <mass value="0.0212636185801172" />
-        <inertia
-          ixx="0"
-          ixy="0"
-          ixz="0"
-          iyy="0"
-          iyz="0"
-          izz="0" />
-      </inertial>
-      <visual>
-        <origin xyz="0 0 0" rpy="0 0 0" />
-        <geometry>
-          <mesh filename="${mounting_plate_visual_mesh}" />
-        </geometry>
-        <material name="${mounting_plate_visual_material_name}">
-          <color rgba="${mounting_plate_visual_material_color}" />
-        </material>
-      </visual>
-      <collision>
-        <origin xyz="0 0 0" rpy="0 0 0" />
-        <geometry>
-          <mesh filename="${mounting_plate_collision_mesh}" />
-        </geometry>
-      </collision>
-    </link>
-    <!-- Link representing the FT300 force-torque sensor -->
-    <link name="${prefix}sensor">
+    <link name="${prefix}robotside">
       <inertial>
         <origin xyz="0.01987 -0.00039088 -0.00013094" rpy="0 0 0" />
@@ -49,5 +19,5 @@
       </inertial>
       <visual>
-        <origin xyz="${-(0.0375 - 0.0027)} 0 0" rpy="0 0 0" />
+        <origin xyz="0 0 0" rpy="0 0 0" />
         <geometry>
           <mesh filename="${sensor_visual_mesh}" />
@@ -58,5 +28,5 @@
       </visual>
       <collision>
-        <origin xyz="${-(0.0375 - 0.0027)} 0 0" rpy="0 0 0" />
+        <origin xyz="0 0 0" rpy="0 0 0" />
         <geometry>
           <mesh filename="${sensor_collision_mesh}" />
@@ -64,9 +34,10 @@
       </collision>
     </link>
-    <!-- Connect force sensor with mounting/coupling plate -->
-    <joint name="${prefix}mounting_plate" type="fixed">
-      <origin xyz="0.0375 0 0" rpy="0 0 0" />
-      <parent link="${prefix}mounting_plate" />
-      <child link="${prefix}sensor" />
+    <link name="${prefix}toolside"/>
+    <link name="${prefix}frame_id"/>
+    <joint name="${prefix}toolside_joint" type="fixed">
+      <origin xyz="0.0348 0 0" rpy="0 0 0" />
+      <parent link="${prefix}robotside" />
+      <child link="${prefix}toolside" />
     </joint>
     <!-- FORCE REFERENCE FRAME
@@ -76,10 +47,9 @@
             points the opposite way away from the connector.
         - The Y axis uses the right hand thumb rule according to X-Z. -->
-    <joint name="${prefix}measurment_joint" type="fixed">
+    <joint name="${prefix}frame_id_joint" type="fixed">
       <origin xyz="0 0 0" rpy="${-pi/2} 0 ${-pi/2}" />
-      <parent link="${prefix}sensor" />
-      <child link="${prefix}ft_frame_id" />
+      <parent link="${prefix}robotside" />
+      <child link="${prefix}frame_id" />
     </joint>
-    <link name="${prefix}ft_frame_id"/>
   </xacro:macro>
 </robot>

File: robotiq_description/urdf/robotiq_fts_300_cpl_062/robotiq_fts_300_cpl_062_common.xacro (robot description, xacro)
@@ -21,9 +21,9 @@
     <xacro:property name="sec_mesh_files" value="${config_visual_parameters['mesh_files']}" />
     <!-- Mesh files -->
-    <xacro:property name="sensor_mesh" value="${sec_mesh_files['sensor']}"/>
-    <xacro:property name="sensor_visual_mesh" value="${sensor_mesh['visual']['mesh']}" scope="parent"/>
-    <xacro:property name="sensor_visual_material_name" value="${sensor_mesh['visual']['material']['name']}" scope="parent"/>
-    <xacro:property name="sensor_visual_material_color" value="${sensor_mesh['visual']['material']['color']}" scope="parent"/>
-    <xacro:property name="sensor_collision_mesh" value="${sensor_mesh['collision']['mesh']}" scope="parent"/>
+    <xacro:property name="mounting_plate_mesh" value="${sec_mesh_files['mounting_plate']}"/>
+    <xacro:property name="mounting_plate_visual_mesh" value="${mounting_plate_mesh['visual']['mesh']}" scope="parent"/>
+    <xacro:property name="mounting_plate_visual_material_name" value="${mounting_plate_mesh['visual']['material']['name']}" scope="parent"/>
+    <xacro:property name="mounting_plate_visual_material_color" value="${mounting_plate_mesh['visual']['material']['color']}" scope="parent"/>
+    <xacro:property name="mounting_plate_collision_mesh" value="${mounting_plate_mesh['collision']['mesh']}" scope="parent"/>
   </xacro:macro>
 </robot>

Commit message: Make ft300 sensor `frame_id` part of the same kinematic tree
The motivation for this change is to make the sensor frame compatible
with some force/compliance controllers that requires all URDF links to
be part of the same kinematic chain.

File: robotiq_description/urdf/robotiq_ft_300/robotiq_ft_300_macro.xacro (robot description, xacro)
@@ -34,11 +34,7 @@
       </collision>
     </link>
+    <!-- Make frame_id link as part of the kinematic change (e.g. for compatibility with cartesian force controllers) -->
+    <link name="${prefix}frame_id"/>
     <link name="${prefix}toolside"/>
-    <link name="${prefix}frame_id"/>
-    <joint name="${prefix}toolside_joint" type="fixed">
-      <origin xyz="0.0348 0 0" rpy="0 0 0" />
-      <parent link="${prefix}robotside" />
-      <child link="${prefix}toolside" />
-    </joint>
     <!-- FORCE REFERENCE FRAME
         As specified in the documentation:
@@ -52,4 +48,10 @@
       <child link="${prefix}frame_id" />
     </joint>
+    <!-- Revert to ROS convention orientation -->
+    <joint name="${prefix}toolside_joint" type="fixed">
+      <origin xyz="0 0 0.0348" rpy="0 ${-pi/2} ${pi/2}" />
+      <parent link="${prefix}frame_id" />
+      <child link="${prefix}toolside" />
+    </joint>
   </xacro:macro>
 </robot>

Commit message: [fix] sensor frame coordinate
The sensor frame is located at the center of the end of the tool side
per the robotiq manual. Wronfully placed at the robot side.

File: robotiq_description/urdf/robotiq_ft_300/robotiq_ft_300_macro.xacro (robot description, xacro)
@@ -44,5 +44,5 @@
         - The Y axis uses the right hand thumb rule according to X-Z. -->
     <joint name="${prefix}frame_id_joint" type="fixed">
-      <origin xyz="0 0 0" rpy="${-pi/2} 0 ${-pi/2}" />
+      <origin xyz="0.0348 0 0" rpy="${-pi/2} 0 ${-pi/2}" />
       <parent link="${prefix}robotside" />
       <child link="${prefix}frame_id" />
@@ -50,5 +50,5 @@
     <!-- Revert to ROS convention orientation -->
     <joint name="${prefix}toolside_joint" type="fixed">
-      <origin xyz="0 0 0.0348" rpy="0 ${-pi/2} ${pi/2}" />
+      <origin xyz="0 0 0" rpy="0 ${-pi/2} ${pi/2}" />
       <parent link="${prefix}frame_id" />
       <child link="${prefix}toolside" />
