Commit message: Rename ambiguous 2f-140 actuating joint name
finger_joint -> left_outer_knuckle_joint

File: robotiq_description/urdf/robotiq_2f_140/inc/robotiq_2f_140_macro.xacro (robot description, xacro)
@@ -210,5 +210,5 @@
         <axis xyz="0 0 1" />
         <limit lower="-3.14" upper="3.14" velocity="2.0" effort="176" />
-        <mimic joint="${prefix}finger_joint" multiplier="${1}" offset="0" />
+        <mimic joint="${prefix}left_outer_knuckle_joint" multiplier="${1}" offset="0" />
       </joint>
     </xacro:macro>
@@ -220,5 +220,5 @@
         <axis xyz="0 0 1" />
         <limit lower="-3.14" upper="3.14" velocity="2.0" effort="176" />
-        <mimic joint="${prefix}finger_joint" multiplier="-1" offset="0" />
+        <mimic joint="${prefix}left_outer_knuckle_joint" multiplier="-1" offset="0" />
       </joint>
     </xacro:macro>
@@ -243,6 +243,7 @@
       <xacro:inner_knuckle prefix="${prefix}" fingerprefix="${fingerprefix}"/>
     </xacro:macro>
-    <xacro:macro name="finger_joint" params="prefix">
-      <joint name="${prefix}finger_joint" type="revolute">
+    <!-- Actuated joint -->
+    <xacro:macro name="left_outer_knuckle_joint" params="prefix">
+      <joint name="${prefix}left_outer_knuckle_joint" type="revolute">
         <origin xyz="0.062905 0.030601 0" rpy="0 ${pi} ${pi}" />
         <parent link="${prefix}base_link" />
@@ -260,5 +261,5 @@
         <axis xyz="0 0 1" />
         <limit lower="-3.14" upper="3.14" velocity="2.0" effort="176" />
-        <mimic joint="${prefix}finger_joint" multiplier="1" offset="0" />
+        <mimic joint="${prefix}left_outer_knuckle_joint" multiplier="1" offset="0" />
       </joint>
       <xacro:finger_joints prefix="${prefix}" fingerprefix="right" reflect="-1.0"/>
@@ -269,5 +270,5 @@
     <xacro:finger_links prefix="${prefix}" fingerprefix="right"/>
     <xacro:tcp prefix="${prefix}"/>
-    <xacro:finger_joint prefix="${prefix}"/>
+    <xacro:left_outer_knuckle_joint prefix="${prefix}"/>
     <xacro:right_outer_knuckle_joint prefix="${prefix}"/>
     <xacro:robotiq_2f_140_transmission prefix="${prefix}"/>

Commit message: Seperate 2f140 fingertip and pads
The fingertip and pads where previously the same entity.

File: robotiq_description/urdf/robotiq_2f_140/inc/robotiq_2f_140_macro.xacro (robot description, xacro)
@@ -1,5 +1,5 @@
 <?xml version="1.0"?>
 <robot xmlns:xacro="http://ros.org/wiki/xacro">
-  <xacro:macro name="robotiq_2f_140" params="prefix visual_parameters_file">
+  <xacro:macro name="robotiq_2f_140" params="prefix visual_parameters_file fingertip_pad_macro_name fingertip_pad_macro_attribute_visual_parameters_file">
     <xacro:include filename="$(find robotiq_description)/urdf/robotiq_2f_140/inc/robotiq_2f_140_transmission.xacro" />
     <xacro:include filename="$(find robotiq_description)/urdf/robotiq_2f_140/inc/robotiq_2f_140_common.xacro" />
@@ -230,4 +230,11 @@
       </joint>
     </xacro:macro>
+    <xacro:macro name="fingertip_pad_joint" params="prefix fingerprefix">
+      <joint name="${prefix}${fingerprefix}_fingertip_pad_joint" type="fixed">
+        <origin xyz="0 0.00476 0 " rpy="0 0 0" />
+        <parent link="${prefix}${fingerprefix}_fingertip" />
+        <child link="${prefix}${fingerprefix}_fingertip_pad" />
+      </joint>
+    </xacro:macro>
     <xacro:macro name="finger_joints" params="prefix fingerprefix reflect">
       <xacro:outer_finger_joint prefix="${prefix}" fingerprefix="${fingerprefix}"/>
@@ -235,4 +242,5 @@
       <xacro:inner_finger_joint prefix="${prefix}" fingerprefix="${fingerprefix}"/>
       <xacro:fingertip_joint prefix="${prefix}" fingerprefix="${fingerprefix}"/>
+      <xacro:fingertip_pad_joint prefix="${prefix}" fingerprefix="${fingerprefix}"/>
     </xacro:macro>
     <xacro:macro name="finger_links" params="prefix fingerprefix">
@@ -242,4 +250,5 @@
       <xacro:fingertip prefix="${prefix}" fingerprefix="${fingerprefix}"/>
       <xacro:inner_knuckle prefix="${prefix}" fingerprefix="${fingerprefix}"/>
+      <xacro:element xacro:name="xacro:${fingertip_pad_macro_name}" prefix="${prefix}${fingerprefix}_" visual_parameters_file="${fingertip_pad_macro_attribute_visual_parameters_file}"/>
     </xacro:macro>
     <!-- Actuated joint -->

File: robotiq_description/urdf/robotiq_2f_140/robotiq_2f_140.xacro (robot description, xacro)
@@ -13,6 +13,9 @@
   -->
   <xacro:include filename="$(find robotiq_description)/urdf/robotiq_2f_140/inc/robotiq_2f_140_macro.xacro" />
+  <xacro:include filename="$(find robotiq_description)/urdf/robotiq_agc_tip_220_140/robotiq_agc_tip_220_140_macro.xacro" />
   <xacro:robotiq_2f_140
     prefix=""
-    visual_parameters_file="$(find robotiq_description)/config/robotiq_2f_140/visual_parameters.yaml"/>
+    visual_parameters_file="$(find robotiq_description)/config/robotiq_2f_140/visual_parameters.yaml"
+    fingertip_pad_macro_name="robotiq_agc_tip_220_140"
+    fingertip_pad_macro_attribute_visual_parameters_file="$(find robotiq_description)/config/robotiq_agc_tip_220_140/visual_parameters.yaml"/>
 </robot>

Commit message: Remove tcp link
Let the user set this link in his xacro top level file.

File: robotiq_description/urdf/robotiq_2f_140/inc/robotiq_2f_140_macro.xacro (robot description, xacro)
@@ -7,13 +7,4 @@
     <xacro:read_model_data
       visual_parameters_file="${visual_parameters_file}"/>
-    <!-- Tool center point origin on the fingertip end when the gripper is fully closed -->
-    <xacro:macro name="tcp" params="prefix">
-      <link name="${prefix}tcp" />
-      <joint name="${prefix}tcp_joint" type="fixed">
-        <origin xyz="0.24127678495 0 0" rpy="0 0 0" />
-        <parent link="${prefix}base_link" />
-        <child link="${prefix}tcp" />
-      </joint>
-    </xacro:macro>
     <xacro:macro name="base_link" params="prefix">
       <link name="${prefix}base_link">
@@ -278,5 +269,4 @@
     <xacro:finger_links prefix="${prefix}" fingerprefix="left"/>
     <xacro:finger_links prefix="${prefix}" fingerprefix="right"/>
-    <xacro:tcp prefix="${prefix}"/>
     <xacro:left_outer_knuckle_joint prefix="${prefix}"/>
     <xacro:right_outer_knuckle_joint prefix="${prefix}"/>
